File: circuit/design/solar_charger.kicad_sch (KiCad schematic)
At the start: 24 parts, among them J1 Screw_Terminal_01x02, J2 USB_A, SW1 SW_SPST, U1 MT3608, U2 TP4056, U3 DW01, U4 FS8205A

Commit message: Backup everything
Parts:
- removed C1, C5: 0.1uF, symbol Device:C
- removed C2, C3: 22uF, symbol Device:C
- removed C4: 10uF, symbol Device:C
- removed D1: BLUE, symbol Device:LED
- removed D2: RED, symbol Device:LED
- removed D3: D_Schottky, symbol Device:D_Schottky
- removed L1: 22uH, symbol pspice:INDUCTOR
- removed R1, R2, R6: 1k, symbol Device:R
- removed R3: 22k, symbol Device:R
- removed R4: 3k, symbol Device:R
- removed R5: 1.2k, symbol Device:R
- removed R7: 100, symbol Device:R
- removed R8: 0, symbol Device:R
- removed SW1: SW_SPST, symbol Switch:SW_SPST
- removed U1: MT3608, Package_TO_SOT_SMD:SOT-23-6, symbol Regulator_Switching:MT3608
- removed U2: TP4056, Package_SO:SOIC-8-1EP_3.9x4.9mm_P1.27mm_EP2.29x3mm, symbol TP4056:TP4056
- removed U3: DW01, Package_TO_SOT_SMD:SOT-23-6_Handsoldering, symbol DW01:DW01
- removed U4: FS8205A, Package_TO_SOT_SMD:SOT-23-6_Handsoldering, symbol FS8205:FS8205A
- added BT1: Battery_Cell, Battery_Holder:BatteryHolder_18650, symbol Device:Battery_Cell
- added J4, J5: Screw_Terminal_01x02, Connector_PinHeader_1.00mm:PinHeader_1x02_P1.00mm_Vertical, symbol Connector:Screw_Terminal_01x02
- added SW2: SW_SPST, Connector_PinHeader_1.00mm:PinHeader_1x02_P1.00mm_Vertical, symbol Switch:SW_SPST
- added U5: TP4056_Breakout, TP4056:TP4056-Module, symbol TP4056_Breakout:TP4056_Breakout
- added U6, U7: MT3608_Breakout, MT3608:MT3608-Module, symbol MT3608_Breakout:MT3608_Breakout
- J1: footprint (none) -> Connector_Molex:Molex_KK-254_AE-6410-02A_1x02_P2.54mm_Vertical
- J2: footprint (none) -> USB_A:USB_A_Breakout
Connections:
- net Earth: no longer names the net of J2.4 (GND)
- net Earth: now also U6.4 (OUT^{-}); no longer J1.1 (Pin_1)
- net VIN renamed V_{IN}
- net V_{IN}: now also U7.1 (IN^{+})
- net VOUT: no longer names the net of J2.1 (VBUS)
- net VOUT: now also U6.3 (OUT^{+})
- new net: J5.2 (Pin_2), U6.1 (IN^{+})
- new net: U5.1 (IN), U7.3 (OUT^{+})
- new net: U5.2 (GND), U7.4 (OUT^{-})
- new net: BT1.1 (+), U5.3 (BAT^{+})
- new net: BT1.2 (-), U5.4 (BAT^{-})
- new net: U5.6 (OUT^{-}), U6.2 (IN^{-})
- new net: J4.1 (Pin_1), SW2.1 (A)
- new net: J4.2 (Pin_2), SW2.2 (B)
- new net GND: J1.1 (Pin_1), U7.2 (IN^{-})
- new net SW_SPST: J5.1 (Pin_1), U5.5 (OUT^{+})
- no-connect marks 6 -> 3
Other:
- added sheet components' module (modules.kicad_sch)
- note added: "Main Circuit"
- note added: "Switch Board"
- note removed: "Battery Charging Controller"
- note removed: "Boost Converter 5V"
- note removed: "USB A Adapter"
